File: hw/pandore-mdot2.kicad_sch (KiCad schematic)
At the start: 42 parts, among them J13 NGFF_M.2_M, J19 NGFF_M.2_AE, M2AE30 M2, M2M110 M2, M2M42 M2, M2M60 M2, M2M80 M2

Commit message: added bringup document and generated ibom to help in manual assembly process
Parts:
- J19: Link - -> https://www.te.com/en/product-2199230-2.html; MFG - -> TE; MPN - -> 2199230-2; now in the parts list
Changed lines of the file:
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@@
 		(body_style 1)
 		(exclude_from_sim no)
-		(in_bom no)
+		(in_bom yes)
 		(on_board yes)
 		(in_pos_files yes)
@@
 			)
 		)
-		(property "Datasheet" "-"
+		(property "Datasheet" "https://www.te.com/commerce/DocumentDelivery/DDEController?Action=srchrtrv&DocNm=2199230&DocType=Customer%20Drawing&DocLang=English&PartCntxt=2199230-2&DocFormat=pdf"
 			(at 135.89 264.16 0)
 			(hide yes)
@@
 			)
 		)
-		(property "MPN" "-"
+		(property "MPN" "2199230-2"
 			(at 135.89 257.81 0)
 			(hide yes)
@@
 			)
 		)
-		(property "MFG" "-"
+		(property "MFG" "TE"
 			(at 154.305 257.81 0)
 			(hide yes)
@@
 			)
 		)
-		(property "Link" "-"
+		(property "Link" "https://www.te.com/en/product-2199230-2.html"
 			(at 173.99 257.81 0)
 			(hide yes)
